File: ir_send_mod.sch (KiCad schematic (older format))
At the start: 25 parts, among them J1 Conn_01x03_Female, J2 Conn_01x05_Male, Q1 2N7000, Q2 IRF9024N, SW1 SW_Coded_SH-7040, SW2 SW_DIP_x04, SW3 SW_SPDT, SW4 SW_SPDT, U1 PIC12F629-IP

Commit message: Update: fix pcb size
Parts:
- renumbered J2 to J1, J1 to J2, R9 to R10, R10 to R11, R11 to R4, R4 to R5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
Connections:
- net labels added: 5V
- wire segments 101 -> 104
